Commit message: undid rename, it wasn't the fix to hte problem i was having with moveit, minor renaming to packages

File: sw_arm_desc/urdf/arm_three.urdf (robot description, URDF)
Before this commit: robot arm_three, 8 links, 7 joints
Links:
- link link_0: geometry collision mesh filename=package://sw_arm_desc/meshes/visual/link_0.STL; visual mesh filename=package://sw_arm_desc/meshes/visual/link_0.STL
- link link_1: geometry collision mesh filename=package://sw_arm_desc/meshes/visual/link_1.STL; visual mesh filename=package://sw_arm_desc/meshes/visual/link_1.STL
- link link_2: geometry collision mesh filename=package://sw_arm_desc/meshes/visual/link_2.STL; visual mesh filename=package://sw_arm_desc/meshes/visual/link_2.STL
- link link_3: geometry collision mesh filename=package://sw_arm_desc/meshes/visual/link_3.STL; visual mesh filename=package://sw_arm_desc/meshes/visual/link_3.STL
- link link_4: geometry collision mesh filename=package://sw_arm_desc/meshes/visual/link_4.STL; visual mesh filename=package://sw_arm_desc/meshes/visual/link_4.STL
- link link_5: geometry collision mesh filename=package://sw_arm_desc/meshes/visual/link_5.STL; visual mesh filename=package://sw_arm_desc/meshes/visual/link_5.STL
- link link_6: geometry collision mesh filename=package://sw_arm_desc/meshes/visual/link_6.STL; visual mesh filename=package://sw_arm_desc/meshes/visual/link_6.STL

Commit message: Fixed bounds on arm joint movements, still uncentered but that doesn't really matter

File: sw_arm_desc/urdf/arm_three.urdf (robot description, URDF)
Before this commit: robot arm_three, 8 links, 7 joints
Joints:
- joint joint_1: limit lower=-1.57 upper=1.570 effort=1000 velocity=1000 -> lower=-2 upper=2 effort=1000 velocity=1000
- joint joint_2: limit lower=-1.57 upper=1.570 effort=1000 velocity=1000 -> lower=-1.160 upper=0.535 effort=1000 velocity=1000
- joint joint_3: limit lower=-1.57 upper=1.570 effort=1000 velocity=1000 -> lower=-2.65 upper=0.625 effort=1000 velocity=1000
- joint joint_5: limit lower=-1.57 upper=1.570 effort=1000 velocity=1000 -> lower=-3.8 upper=0.232 effort=1000 velocity=1000

Commit message: Changed URDF to use collision meshes for collision, though both STL's are identical for now...

File: sw_arm_desc/urdf/arm_three.urdf (robot description, URDF)
Before this commit: robot arm_three, 8 links, 7 joints
Links:
- link link_0: geometry collision mesh filename=package://sw_arm_desc/meshes/collision/link_0.STL; visual mesh filename=package://sw_arm_desc/meshes/visual/link_0.STL
- link link_1: geometry collision mesh filename=package://sw_arm_desc/meshes/collision/link_1.STL; visual mesh filename=package://sw_arm_desc/meshes/visual/link_1.STL
- link link_2: geometry collision mesh filename=package://sw_arm_desc/meshes/collision/link_2.STL; visual mesh filename=package://sw_arm_desc/meshes/visual/link_2.STL
- link link_3: geometry collision mesh filename=package://sw_arm_desc/meshes/collision/link_3.STL; visual mesh filename=package://sw_arm_desc/meshes/visual/link_3.STL
- link link_4: geometry collision mesh filename=package://sw_arm_desc/meshes/collision/link_4.STL; visual mesh filename=package://sw_arm_desc/meshes/visual/link_4.STL
- link link_5: geometry collision mesh filename=package://sw_arm_desc/meshes/collision/link_5.STL; visual mesh filename=package://sw_arm_desc/meshes/visual/link_5.STL
- link link_6: geometry collision mesh filename=package://sw_arm_desc/meshes/collision/link_6.STL; visual mesh filename=package://sw_arm_desc/meshes/visual/link_6.STL
Joints:
- joint joint_1: limit lower=-2 upper=2 effort=1000 velocity=1000 -> lower=-2 upper=2 effort=1000.0 velocity=1000.0
- joint joint_2: limit lower=-1.160 upper=0.535 effort=1000 velocity=1000 -> lower=-1.160 upper=0.535 effort=1000.0 velocity=1000.0
- joint joint_3: limit lower=-2.65 upper=0.625 effort=1000 velocity=1000 -> lower=-2.65 upper=0.625 effort=1000.0 velocity=1000.0
- joint joint_4: limit lower=-1.57 upper=1.570 effort=1000 velocity=1000 -> lower=-1.57 upper=1.570 effort=1000.0 velocity=1000.0
- joint joint_5: limit lower=-3.8 upper=0.232 effort=1000 velocity=1000 -> lower=-3.8 upper=0.232 effort=1000.0 velocity=1000.0
- joint joint_6: limit lower=-1.57 upper=1.570 effort=1000 velocity=1000 -> lower=-1.57 upper=1.570 effort=1000.0 velocity=1000.0
