Commit message: Joint limits roughly good enough hopefully

File: sw_arm_desc/urdf/arm_final.urdf (robot description, URDF)
Before this commit: robot arm_final, 8 links, 7 joints
Joints:
- removed joint world_to_link_zero
- added joint world_to_link_0: type fixed, parent world, child link_0, origin xyz=0 0 0.001 rpy=0 0 0
- joint joint_1: limit lower=0 upper=0 effort=0 velocity=0 -> lower=-1.52 upper=1.52 effort=1000.0 velocity=1000.0
- joint joint_2: limit lower=0 upper=0 effort=0 velocity=0 -> lower=-1.8 upper=0 effort=1000.0 velocity=1000.0
- joint joint_3: limit lower=0 upper=0 effort=0 velocity=0 -> lower=-0.75 upper=2.59 effort=1000.0 velocity=1000.0
- joint joint_4: limit lower=0 upper=0 effort=0 velocity=0 -> lower=-2.0 upper=3.0 effort=1000.0 velocity=1000.0
- joint joint_5: limit lower=0 upper=0 effort=0 velocity=0 -> lower=-1.084 upper=1.0 effort=1000.0 velocity=1000.0
- joint joint_6: limit lower=0 upper=0 effort=0 velocity=0 -> lower=-1.52 upper=1.52 effort=1000.0 velocity=1000.0
