Commit message: Made a new URDF with a fake gripper

File: arm_moveit_config/config/arm_three.ros2_control.xacro (robot description, xacro)
@@ -6,5 +6,7 @@
             <hardware>
                 <!-- By default, set up controllers for simulation. This won't work on real hardware -->
-                <plugin>mock_components/GenericSystem</plugin>
+                <!-- by NOT default, I'm gonna tell this to use gazebo -->
+                <!-- <plugin>mock_components/GenericSystem</plugin> -->
+                <plugin>gazebo_ros2_control/GazeboSystem</plugin>
             </hardware>
             <joint name="joint_1">
@@ -57,4 +59,12 @@
             </joint>
         </ros2_control>
+        <gazebo>
+            <plugin name="gazebo_ros2_control" filename="libgazebo_ros2_control">
+                <!-- when gazebo fires up gazebo_ros2_control plugin, use this config -->
+                <parameters>
+                    $(find arm_moveit_config)/config/ros2_control.yaml
+                </parameters>
+            </plugin>
+        </gazebo>
     </xacro:macro>
 </robot>

File: sw_arm_desc/urdf/arm_end_effector.urdf (robot description, URDF)
Before this commit: robot arm_end_effector.urdf, 9 links, 8 joints
Links:
- added link gripper_link_slave, mass 0.28883; collision box size=0.1 0.025 0.025; visual box size=0.1 0.025 0.025
Joints:
- added joint grip_joint_slave: type prismatic, parent link_6_fake, child gripper_link_slave, origin xyz=0.025 -0.025 0, axis 0 1 0, limit lower=-0.0125 upper=0.025 effort=1000.0 velocity=1000.0, mimic joint=grip_joint multiplier=-1 offset=0
- joint grip_joint: limit lower=-0.25 upper=0.25 effort=1000.0 velocity=1000.0 -> lower=-0.0125 upper=0.025 effort=1000.0 velocity=1000.0
