Commit message: Arm working with fake end effector and moveit motion planning verified

File: arm_moveit_config/config/arm_end_effector.ros2_control.xacro (robot description, xacro)
@@ -1,12 +1,10 @@
 <?xml version="1.0"?>
 <robot xmlns:xacro="http://www.ros.org/wiki/xacro">
-    <xacro:macro name="arm_three_ros2_control" params="name initial_positions_file">
+    <xacro:macro name="arm_end_effector_ros2_control" params="name initial_positions_file">
         <xacro:property name="initial_positions" value="${load_yaml(initial_positions_file)['initial_positions']}"/>
         <ros2_control name="${name}" type="system">
             <hardware>
                 <!-- By default, set up controllers for simulation. This won't work on real hardware -->
-                <!-- by NOT default, I'm gonna tell this to use gazebo -->
-                <!-- <plugin>mock_components/GenericSystem</plugin> -->
-                <plugin>gazebo_ros2_control/GazeboSystem</plugin>
+                <plugin>mock_components/GenericSystem</plugin>
             </hardware>
             <joint name="joint_1">
@@ -58,13 +56,13 @@
                 <state_interface name="velocity"/>
             </joint>
+            <joint name="grip_joint">
+                <command_interface name="position"/>
+                <command_interface name="velocity"/>
+                <state_interface name="position">
+                  <param name="initial_value">${initial_positions['grip_joint']}</param>
+                </state_interface>
+                <state_interface name="velocity"/>
+            </joint>
         </ros2_control>
-        <gazebo>
-            <plugin name="gazebo_ros2_control" filename="libgazebo_ros2_control">
-                <!-- when gazebo fires up gazebo_ros2_control plugin, use this config -->
-                <parameters>
-                    $(find arm_moveit_config)/config/ros2_control.yaml
-                </parameters>
-            </plugin>
-        </gazebo>
     </xacro:macro>
 </robot>
