Commit message: ros being dumb

File: arm_motor_controller/config/armtest.ros2_control.xacro (robot description, xacro)
@@ -47,5 +47,5 @@
                 <state_interface name="velocity"/>
             </joint>
-            <joint name="joint_6">
+            <!-- <joint name="joint_6">
                 <command_interface name="position"/>
                 <command_interface name="velocity"/>
@@ -54,5 +54,5 @@
                 </state_interface>
                 <state_interface name="velocity"/>
-            </joint>
+            </joint> -->
         </ros2_control>
     </xacro:macro>

File: arm_moveit_config/config/arm_three.ros2_control.xacro (robot description, xacro)
@@ -6,7 +6,9 @@
             <hardware>
                 <!-- By default, set up controllers for simulation. This won't work on real hardware -->
-                <plugin>mock_components/GenericSystem</plugin>
+                <plugin>arm_motor_controller/ArmSystemHardware</plugin>
             </hardware>
             <joint name="joint_1">
+                <param name="type">iCL</param>
+                <param name="id">1</param>
                 <command_interface name="position"/>
                 <command_interface name="velocity"/>
@@ -17,4 +19,6 @@
             </joint>
             <joint name="joint_2">
+                <param name="type">iCL</param>
+                <param name="id">2</param>
                 <command_interface name="position"/>
                 <command_interface name="velocity"/>
@@ -25,4 +29,6 @@
             </joint>
             <joint name="joint_3">
+                <param name="type">iCL</param>
+                <param name="id">3</param>
                 <command_interface name="position"/>
                 <command_interface name="velocity"/>
@@ -33,4 +39,6 @@
             </joint>
             <joint name="joint_4">
+                <param name="type">iCL</param>
+                <param name="id">4</param>
                 <command_interface name="position"/>
                 <command_interface name="velocity"/>
@@ -41,4 +49,6 @@
             </joint>
             <joint name="joint_5">
+                <param name="type">iCL</param>
+                <param name="id">5</param>
                 <command_interface name="position"/>
                 <command_interface name="velocity"/>
@@ -49,4 +59,6 @@
             </joint>
             <joint name="joint_6">
+                <param name="type">iCL</param>
+                <param name="id">6</param>
                 <command_interface name="position"/>
                 <command_interface name="velocity"/>

Commit message: It launches.

File: arm_motor_controller/config/armtest.ros2_control.xacro (robot description, xacro)
@@ -18,5 +18,5 @@
             </joint>
             <joint name="joint_2">
-                <param name="type">iCL</param>
+                <param name="type">none</param>
                 <param name="id">2</param>
                 <command_interface name="position"/>
@@ -28,5 +28,5 @@
             </joint>
             <joint name="joint_3">
-                <param name="type">iCL</param>
+                <param name="type">none</param>
                 <param name="id">3</param>
                 <command_interface name="position"/>
@@ -38,5 +38,5 @@
             </joint>
             <joint name="joint_4">
-                <param name="type">iCL</param>
+                <param name="type">none</param>
                 <param name="id">4</param>
                 <command_interface name="position"/>
@@ -48,5 +48,5 @@
             </joint>
             <joint name="joint_5">
-                <param name="type">iCL</param>
+                <param name="type">none</param>
                 <param name="id">5</param>
                 <command_interface name="position"/>
@@ -57,5 +57,7 @@
                 <state_interface name="velocity"/>
             </joint>
-            <!-- <joint name="joint_6">
+            <joint name="joint_6">
+                <param name="type">none</param>
+                <param name="id">6</param>
                 <command_interface name="position"/>
                 <command_interface name="velocity"/>
@@ -64,5 +66,15 @@
                 </state_interface>
                 <state_interface name="velocity"/>
-            </joint> -->
+            </joint>
+            <joint name="grip_joint">
+                <param name="type">none</param>
+                <param name="id">7</param>
+                <command_interface name="position"/>
+                <command_interface name="velocity"/>
+                <state_interface name="position">
+                  <param name="initial_value">${initial_positions['grip_joint']}</param>
+                </state_interface>
+                <state_interface name="velocity"/>
+            </joint>
         </ros2_control>
     </xacro:macro>

File: arm_motor_controller/config/armtest.urdf.xacro (robot description, xacro)
@@ -1,7 +1,7 @@
 <?xml version="1.0"?>
-<robot xmlns:xacro="http://www.ros.org/wiki/xacro" name="armtest">
+<robot xmlns:xacro="http://www.ros.org/wiki/xacro" name="arm_end_effector">
     <xacro:arg name="initial_positions_file" default="initial_positions.yaml" />
     <!-- Import arm_three urdf file -->
-    <xacro:include filename="$(find sw_arm_desc)/urdf/arm_three.urdf" />
+    <xacro:include filename="$(find sw_arm_desc)/urdf/arm_end_effector.urdf" />
     <!-- Import control_xacro -->
     <xacro:include filename="armtest.ros2_control.xacro" />
