Commit message: Working code for arm so far

File: arm_pkg/urdf/final_hw.ros2_control.xacro (robot description, xacro)
@@ -15,9 +15,12 @@
             <joint name="joint_1">
                 <param name="type">iCL</param>
+                <!-- <param name="type">none</param> -->
                 <param name="id">1</param>
-                <param name="min">-32000</param>
-                <param name="max">32000</param>
+                <param name="min">0</param>
+                <param name="max">306000</param>
                 <param name="rpm">64</param>
-                <param name="homePosition">0</param>
+                <param name="homeSpeed">50</param>
+                <param name="homeConfig">2</param>
+                <param name="reverse">0</param>
                 <command_interface name="position"/>
                 <command_interface name="velocity"/>
@@ -30,10 +33,13 @@
             </joint>
             <joint name="joint_2">
+                <!-- <param name="type">iCL</param> -->
                 <param name="type">none</param>
                 <param name="id">2</param>
                 <param name="min">0</param>
-                <param name="max">3200</param>
+                <param name="max">82000</param>
                 <param name="rpm">32</param>
-                <param name="homePosition">0</param>
+                <param name="homeSpeed">5</param>
+                <param name="homeConfig">2</param>
+                <param name="reverse">0</param>
                 <command_interface name="position"/>
                 <command_interface name="velocity"/>
@@ -46,11 +52,13 @@
             </joint>
             <joint name="joint_3">
-                <param name="type">none</param>
-                <!-- <param name="type">iCL</param> -->
+                <param name="type">iCL</param>
+                <!-- <param name="type">none</param> -->
                 <param name="id">3</param>
-                <param name="min">-32000</param>
+                <param name="min">-310000</param>
                 <param name="max">0</param>
                 <param name="rpm">32</param>
-                <param name="reverse">1</param>
+                <param name="homeSpeed">10</param>
+                <param name="homeConfig">19</param>
+                <param name="reverse">0</param>
                 <command_interface name="position"/>
                 <command_interface name="velocity"/>
@@ -63,10 +71,13 @@
             </joint>
             <joint name="joint_4">
-                <param name="type">none</param>
+                <param name="type">iCL</param>
+                <!-- <param name="type">none</param> -->
                 <param name="id">4</param>
                 <param name="min">0</param>
-                <param name="max">3200</param>
+                <param name="max">176000</param>
                 <param name="rpm">32</param>
-                <param name="homePosition">0</param>
+                <param name="homeSpeed">10</param>
+                <param name="homeConfig">2</param>
+                <param name="reverse">1</param>
                 <command_interface name="position"/>
                 <command_interface name="velocity"/>
@@ -84,5 +95,7 @@
                 <param name="max">3200</param>
                 <param name="rpm">32</param>
-                <param name="homePosition">0</param>
+                <param name="homeSpeed">0</param>
+                <param name="homeConfig">0</param>
+                <param name="reverse">0</param>
                 <command_interface name="position"/>
                 <command_interface name="velocity"/>
@@ -102,5 +115,7 @@
                 <param name="max">288000</param>
                 <param name="rpm">2400</param>
-                <param name="homePosition">0</param>
+                <param name="homeSpeed">0</param>
+                <param name="homeConfig">0</param>
+                <param name="reverse">0</param>
                 <command_interface name="position"/>
                 <command_interface name="velocity"/>

File: sw_arm_desc/urdf/arm_final_sim.urdf (robot description, URDF)
Before this commit: robot arm_final, 10 links, 9 joints
Joints:
- joint joint_1: limit lower=-1.52 upper=1.52 effort=1000.0 velocity=1000.0 -> lower=-2.094 upper=1.57 effort=1000.0 velocity=1000.0
